File: VCO-3340.kicad_sch (KiCad schematic)
At the start: 118 parts, among them J1 AudioJack2, J10 Conn_01x01, J11 Conn_01x01, J12 Conn_01x01, J13 Conn_01x01, J14 Conn_01x01, J15 Conn_01x01, J16 Conn_01x01, J17 Conn_01x01, J18 Conn_01x01, J19 Conn_01x01, J2 AudioJack2, J20 Conn_01x01, J21 Conn_01x01, J22 Conn_01x01, J23 Conn_01x01, J24 Conn_01x01, J3 AudioJack2, J4 AudioJack2, J5 AudioJack2, J6 Conn_01x01, J7 Conn_01x01, J8 Conn_02x05_Odd_Even, J9 Conn_01x01, U1 TL074, U2 AS3340, U3 TL074, U4 LM311, U5 4013, U6 LM79L05_TO92, U7 LM78L05_TO92

Commit message: small tweaks
Parts:
- C9: value 10p -> 100p
Changed lines of the file:
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@@
 			)
 		)
-		(property "Value" "10p"
+		(property "Value" "100p"
 			(at 359.41 135.89 90)
 			(show_name no)

Commit message: compensation caps
Parts:
- added C22, C23, C24, C25, C26: 100p, Capacitor_THT:C_Disc_D5.1mm_W3.2mm_P5.00mm, symbol Device:C
- C9: value 100p -> 22p
Connections:
- net SAW_OUT: now also C23.2
- net SQ_OUT: now also C25.2
- net SUB_OUT: now also C26.2
- net TR_OUT: now also C24.2
- net at R12.2, R13.2, R17.1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: now also C22.1
- net at R17.2, R20.2, U1.8: now also C22.2
- net at R23.2, R26.1, R29.1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: now also C24.1
- net at R34.2, R35.1, R36.1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: now also C26.1
- net at R22.2, R25.1, R28.1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: now also C23.1
- net at R31.2, R32.1, R33.1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: now also C25.1
Other:
- moved on the sheet: U1B, U1C, U3A, U3B, U3D

Commit message: Use 5V regulator to generate offsets
Parts:
- removed C21: 1u, Capacitor_THT:CP_Radial_D6.3mm_P2.50mm, symbol Device:C_Polarized
- removed C26: 100p, Capacitor_THT:C_Disc_D5.1mm_W3.2mm_P5.00mm, symbol Device:C
- removed RV10, RV11, RV14, RV16: 10k, Potentiometer_THT:Potentiometer_Bourns_3296Y_Vertical, symbol Device:R_Potentiometer_Trim
- added C9: 0.1u, Capacitor_THT:C_Disc_D5.1mm_W3.2mm_P5.00mm, symbol Device:C
- C25: value 100p -> 0.1u
- R1: value 22k -> 20k
- R10, R26, R29: value 220k -> 200k
- R23: value 110k -> 100k
- R30: value 4.7k -> 1k
- R31: value 100k -> 18k
- R32: value 100k -> 36k
- R33: value 91k -> 36k
- R34: value 100k -> 10k
- R35: value 100k -> 20k
- R36: value 82k -> 20k
- renumbered C8 to C10, C23 to C11, C24 to C12, C9 to C13, C10 to C14, C11 to C15, C12 to C16, C13 to C17, C14 to C18, C15 to C19, C16 to C20, C17 to C21, C18 to C22, C19 to C23, C20 to C24, C22 to C8, RV12 to RV10, RV13 to RV11, RV15 to RV12, RV17 to RV13
Connections:
- net +12V: no longer C24.1, R30.2, U5.14 (VDD)
- net +5V: now also C24.1, C25.1, R30.2, U5.14 (VDD)
- net -5V: now also R25.2, R26.2, R32.2, R35.2, C9.1
- net GND: now also C25.2, C9.2
- net SQ_OUT: no longer C25.2
- net at R31.2, R32.1, R33.1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: no longer C25.1
Other:
- moved on the sheet: R25, R26, R31, R32, R33, R35, RV12, U1B, U3A
